File: pcb_design/vitimonitor_sensor/user_itf.kicad_sch (KiCad schematic)
At the start: 0 parts

Commit message: Schematic update, hierarchical approach done, missing SX1261
Parts:
- added C3: 1u, symbol Device:C_Small
- added D1, D5: ESD3V3, Diode_SMD:D_SOD-923, symbol Diode:ESD9B3.3ST5G
- added D7: GREEN, symbol Device:LED_Small
- added R7: 10k, symbol Device:R_Small
- added R8: 1k, symbol Device:R_Small
- added SW3: BOOT, symbol Switch:SW_SPST
- added SW4: RESETN, symbol Switch:SW_SPST
Connections:
- new net: D7.2 (A), R8.2
- new net +3.3V: R7.1, R8.1
- new net BOOT: D1.2 (A2), SW3.2 (B)
- new net EN: C3.1, D5.2 (A2), R7.2, SW4.2 (B)
- new net GND: C3.2, D1.1 (A1), D5.1 (A1), D7.1 (K), SW3.1 (A), SW4.1 (A)
Other:
- note added: "3V3 OK"
- note added: "USER INTERFACE"
