File: pcb_design/vitimonitor_sensor/connectors.kicad_sch (KiCad schematic)
At the start: 0 parts

Commit message: Schematic update, hierarchical approach done, missing SX1261
Parts:
- added J1, J3: Conn_01x04, symbol Connector_Generic:Conn_01x04
- added J10: Conn_01x10, symbol Connector_Generic:Conn_01x10
- added J9: Pin_2x5, symbol Connector_Generic:Conn_02x05_Odd_Even
- added R4, R6: 2.2k, symbol Device:R_Small
Connections:
- new net +3.3V: J1.1 (Pin_1), J10.10 (Pin_10), J3.1 (Pin_1), J9.1 (Pin_1), J9.2 (Pin_2), R4.1, R6.1
- new net +BATT: J10.6 (Pin_6)
- new net 5V_OK: J10.5 (Pin_5)
- new net BOOT: J10.8 (Pin_8)
- new net CLK: J9.4 (Pin_4)
- new net CS: J9.6 (Pin_6)
- new net EN: J10.9 (Pin_9)
- new net GND: J1.4 (Pin_4), J10.2 (Pin_2), J3.4 (Pin_4), J9.10 (Pin_10), J9.9 (Pin_9)
- new net IRQ: J9.8 (Pin_8)
- new net MISO: J9.5 (Pin_5)
- new net MOSI: J9.7 (Pin_7)
- new net RESET: J9.3 (Pin_3)
- new net SCL: J1.2 (Pin_2), R4.2
- new net SDA: J1.3 (Pin_3), R6.2
- new net UART_RX: J3.3 (Pin_3)
- new net UART_TX: J3.2 (Pin_2)
- new net USB_D+: J10.3 (Pin_3)
- new net USB_D-: J10.4 (Pin_4)
- new net VBAT_OK: J10.7 (Pin_7)
- new net VBUS_OK: J10.1 (Pin_1)
Other:
- note added: "I2C CONNECTOR"
- note added: "MAIN SIGNALS CONNECTOR"
- note added: "SPI CONNECTOR"
- note added: "UART CONNECTOR"

Commit message: Changes due to a first review
Parts:
- added C4: 100n, symbol Device:C_Small
- added D2: ESD3V3, Diode_SMD:D_SOD-923, symbol Diode:ESD9B3.3ST5G
- added F1: Polyfuse, symbol Device:Polyfuse
- added J2: USB_C_Receptacle_USB2.0_14P, symbol Connector:USB_C_Receptacle_USB2.0_14P
- added R10, R9: 5.1k, symbol Device:R_Small
- added R3: 100k, symbol Device:R_Small
- added U1: USBLC6-2SC6, Package_TO_SOT_SMD:SOT-23-6, symbol Power_Protection:USBLC6-2SC6
Connections:
- net GND: now also C4.2, D2.1 (A1), J2.A1 (GND), J2.A12 (GND), J2.B1 (GND), J2.B12 (GND), J2.S1 (SHIELD), R10.2, R3.1, R9.2, U1.2 (GND)
- net USB_D+: now also U1.6 (I/O1)
- net USB_D-: now also U1.4 (I/O2)
- net VBUS_OK: now also C4.1, D2.2 (A2), F1.2, U1.5 (VBUS)
- new net: F1.1, J2.A4 (VBUS), J2.A9 (VBUS), J2.B4 (VBUS), J2.B9 (VBUS), R3.2
- new net CC1: J2.A5 (CC1), R9.1
- new net CC2: J2.B5 (CC2), R10.1
- new net D+: J2.A6 (D+), J2.B6 (D+), U1.1 (I/O1)
- new net D-: J2.A7 (D-), J2.B7 (D-), U1.3 (I/O2)
Other:
- note added: "ESD da cambiare a 5V !!!!!!!!"
- note added: "USB-C"
- moved on the sheet: J1, J10, J3, J9, R4, R6
