File: pcb_design/vitimonitor_sensor/power.kicad_sch (KiCad schematic)
At the start: 28 parts, among them J7 USB_C_Receptacle_USB2.0_14P, J8 Conn_01x02, Q1 Si2371EDS, U4 USBLC6-2SC6, U6 BQ24075RGT, U7 LM1117DT-3.3

Commit message: Changes due to a first review
Parts:
- removed C11: 100n, symbol Device:C_Small
- removed D6: ESD3V3, Diode_SMD:D_SOD-923, symbol Diode:ESD9B3.3ST5G
- removed F2: Polyfuse, symbol Device:Polyfuse
- removed J7: USB_C_Receptacle_USB2.0_14P, symbol Connector:USB_C_Receptacle_USB2.0_14P
- removed R17, R18: 5.1k, symbol Device:R_Small
- removed R19: 100k, symbol Device:R_Small
- removed U4: USBLC6-2SC6, Package_TO_SOT_SMD:SOT-23-6, symbol Power_Protection:USBLC6-2SC6
- R20, R21: value 1.1k -> 110k
Other:
- note added: "1% per essere preciso"
- note added: "Aggiungi 100n su OUT per RF alte -> 100n più vicino a OUT rispetto a 22u"
- note added: "Check DIODO affinche vbatt < di Vcatodo diodo => 1N4007"
- note removed: "USB-C"
- moved on the sheet: C13, C14, C15, D10, D9, R22, R23, R24, R25, R26, U6
